Commit message: serial bridge for arduino to pi communication

File: ros2_ws/src/description/urdf/warehouse_bot.urdf.xacro (robot description, xacro)
@@ -1,37 +1,68 @@
 <?xml version="1.0"?>
+<!--
+  warehouse_bot.urdf.xacro
+  ========================
+  4-wheel differential drive (skid steer) robot
+  Real hardware measurements as of current build.
+  Coordinate frame: REP-103
+    x = forward, y = left, z = up
+    base_link origin at geometric center of chassis, at ground level
+  TF tree:
+    base_link
+      ├── front_left_wheel_link
+      ├── front_right_wheel_link
+      ├── rear_left_wheel_link
+      ├── rear_right_wheel_link
+      ├── base_laser        (LiDAR)
+      ├── camera_link       (placeholder)
+      └── imu_link          (IMU)
+-->
 <robot name="warehouse_bot" xmlns:xacro="http://www.ros.org/wiki/xacro">
   <!-- ============================================================
-       warehouse_bot.urdf.xacro
-       Minimal differential drive robot for warehouse delivery bot.
-       Chassis: 0.4m x 0.3m x 0.15m box
-       Drive:   4 wheels (2 driven, 2 caster)
-       Sensors: 2D LiDAR (top center), Camera (front face)
-       ============================================================ -->
-  <!-- ==================== PROPERTIES ==================== -->
+       PROPERTIES
+       ============================================================ -->
   <!-- Chassis -->
-  <xacro:property name="chassis_length" value="0.4"/>
-  <xacro:property name="chassis_width"  value="0.3"/>
-  <xacro:property name="chassis_height" value="0.15"/>
-  <xacro:property name="chassis_mass"   value="5.0"/>
-  <!-- Drive wheels -->
-  <xacro:property name="wheel_radius"   value="0.05"/>
-  <xacro:property name="wheel_width"    value="0.04"/>
-  <xacro:property name="wheel_mass"     value="0.5"/>
-  <xacro:property name="wheel_y_offset" value="0.17"/>  <!-- half chassis_width + half wheel_width -->
-  <!-- Caster -->
-  <xacro:property name="caster_radius"  value="0.025"/>
-  <xacro:property name="caster_mass"    value="0.1"/>
-  <!-- Sensor offsets -->
-  <xacro:property name="lidar_z_offset"  value="0.10"/>  <!-- above chassis top -->
-  <xacro:property name="camera_x_offset" value="0.21"/>  <!-- front face -->
-  <xacro:property name="camera_z_offset" value="0.05"/>
-  <!-- ==================== INERTIA MACROS ==================== -->
-  <xacro:macro name="box_inertia" params="m x y z">
+  <xacro:property name="chassis_length"  value="0.20"/>
+  <xacro:property name="chassis_width"   value="0.155"/>
+  <xacro:property name="chassis_height"  value="0.065"/>
+  <xacro:property name="chassis_mass"    value="3.0"/>
+  <!-- Wheels -->
+  <xacro:property name="wheel_radius"    value="0.04"/>
+  <xacro:property name="wheel_width"     value="0.035"/>
+  <xacro:property name="wheel_mass"      value="0.3"/>
+  <xacro:property name="wheel_separation" value="0.21"/>   <!-- left to right, center to center -->
+  <xacro:property name="wheelbase"       value="0.095"/>   <!-- front to rear axle, center to center -->
+  <!-- LiDAR -->
+  <xacro:property name="lidar_height"    value="0.28"/>    <!-- from ground -->
+  <xacro:property name="lidar_radius"    value="0.04"/>
+  <xacro:property name="lidar_length"    value="0.06"/>
+  <!-- Derived: chassis sits on top of wheels -->
+  <!-- chassis_z = wheel_radius (ground to axle) + chassis_height/2 -->
+  <xacro:property name="chassis_z"       value="${wheel_radius + chassis_height / 2.0}"/>
+  <!-- ============================================================
+       MATERIALS
+       ============================================================ -->
+  <material name="blue">
+    <color rgba="0.1 0.4 0.8 1.0"/>
+  </material>
+  <material name="dark_grey">
+    <color rgba="0.2 0.2 0.2 1.0"/>
+  </material>
+  <material name="grey">
+    <color rgba="0.5 0.5 0.5 1.0"/>
+  </material>
+  <material name="black">
+    <color rgba="0.1 0.1 0.1 1.0"/>
+  </material>
+  <!-- ============================================================
+       INERTIA MACROS
+       ============================================================ -->
+  <xacro:macro name="box_inertia" params="m l w h">
     <inertial>
       <mass value="${m}"/>
       <inertia
-        ixx="${m*(y*y+z*z)/12}" ixy="0" ixz="0"
-        iyy="${m*(x*x+z*z)/12}" iyz="0"
-        izz="${m*(x*x+y*y)/12}"/>
+        ixx="${m*(w*w+h*h)/12}" ixy="0" ixz="0"
+        iyy="${m*(l*l+h*h)/12}" iyz="0"
+        izz="${m*(l*l+w*w)/12}"/>
     </inertial>
   </xacro:macro>
@@ -45,133 +76,148 @@
     </inertial>
   </xacro:macro>
-  <xacro:macro name="sphere_inertia" params="m r">
-    <inertial>
-      <mass value="${m}"/>
-      <inertia
-        ixx="${2*m*r*r/5}" ixy="0" ixz="0"
-        iyy="${2*m*r*r/5}" iyz="0"
-        izz="${2*m*r*r/5}"/>
-    </inertial>
-  </xacro:macro>
-  <!-- ==================== WHEEL MACRO ==================== -->
-  <xacro:macro name="drive_wheel" params="name y_reflect">
-    <link name="${name}_wheel_link">
+  <!-- ============================================================
+       BASE LINK (chassis)
+       ============================================================ -->
+  <link name="base_link">
+    <xacro:box_inertia m="${chassis_mass}"
+                       l="${chassis_length}"
+                       w="${chassis_width}"
+                       h="${chassis_height}"/>
+    <visual>
+      <origin xyz="0 0 ${chassis_z}" rpy="0 0 0"/>
+      <geometry>
+        <box size="${chassis_length} ${chassis_width} ${chassis_height}"/>
+      </geometry>
+      <material name="blue"/>
+    </visual>
+    <collision>
+      <origin xyz="0 0 ${chassis_z}" rpy="0 0 0"/>
+      <geometry>
+        <box size="${chassis_length} ${chassis_width} ${chassis_height}"/>
+      </geometry>
+    </collision>
+  </link>
+  <!-- ============================================================
+       WHEEL MACRO
+       ============================================================ -->
+  <xacro:macro name="wheel" params="name x_pos y_pos">
+    <link name="${name}_link">
+      <xacro:cylinder_inertia m="${wheel_mass}" r="${wheel_radius}" h="${wheel_width}"/>
       <visual>
-        <geometry><cylinder radius="${wheel_radius}" length="${wheel_width}"/></geometry>
-        <material name="dark_grey"><color rgba="0.2 0.2 0.2 1"/></material>
+        <origin xyz="0 0 0" rpy="${pi/2} 0 0"/>
+        <geometry>
+          <cylinder radius="${wheel_radius}" length="${wheel_width}"/>
+        </geometry>
+        <material name="dark_grey"/>
       </visual>
       <collision>
-        <geometry><cylinder radius="${wheel_radius}" length="${wheel_width}"/></geometry>
+        <origin xyz="0 0 0" rpy="${pi/2} 0 0"/>
+        <geometry>
+          <cylinder radius="${wheel_radius}" length="${wheel_width}"/>
+        </geometry>
       </collision>
-      <xacro:cylinder_inertia m="${wheel_mass}" r="${wheel_radius}" h="${wheel_width}"/>
     </link>
-    <joint name="${name}_wheel_joint" type="continuous">
+    <joint name="${name}_joint" type="continuous">
       <parent link="base_link"/>
-      <child  link="${name}_wheel_link"/>
-      <!-- Wheels are mid-chassis height, rotated 90deg to spin on Y axis -->
-      <origin xyz="0 ${y_reflect * wheel_y_offset} ${-chassis_height/2 + wheel_radius}"
-              rpy="${pi/2} 0 0"/>
-      <axis xyz="0 0 1"/>
+      <child  link="${name}_link"/>
+      <origin xyz="${x_pos} ${y_pos} ${wheel_radius}" rpy="0 0 0"/>
+      <axis xyz="0 1 0"/>
       <dynamics damping="0.1" friction="0.1"/>
     </joint>
+    <!-- Gazebo wheel friction -->
+    <gazebo reference="${name}_link">
+      <mu1>1.0</mu1>
+      <mu2>1.0</mu2>
+      <material>Gazebo/DarkGrey</material>
+    </gazebo>
   </xacro:macro>
-  <!-- ==================== BASE LINK ==================== -->
-  <!-- base_link is the robot's origin at ground level, center of chassis -->
-  <link name="base_link">
-    <visual>
-      <origin xyz="0 0 ${chassis_height/2}"/>
-      <geometry>
-        <box size="${chassis_length} ${chassis_width} ${chassis_height}"/>
-      </geometry>
-      <material name="blue"><color rgba="0.1 0.4 0.8 1"/></material>
+  <!-- ============================================================
+       INSTANTIATE 4 WHEELS
+       front_left, front_right, rear_left, rear_right
+       ============================================================ -->
+  <xacro:wheel name="front_left_wheel"
+               x_pos="${wheelbase/2}"
+               y_pos="${wheel_separation/2}"/>
+  <xacro:wheel name="front_right_wheel"
+               x_pos="${wheelbase/2}"
+               y_pos="${-wheel_separation/2}"/>
+  <xacro:wheel name="rear_left_wheel"
+               x_pos="${-wheelbase/2}"
+               y_pos="${wheel_separation/2}"/>
+  <xacro:wheel name="rear_right_wheel"
+               x_pos="${-wheelbase/2}"
+               y_pos="${-wheel_separation/2}"/>
+  <!-- ============================================================
+       LIDAR LINK (base_laser)
+       Mounted at center of chassis, 0.28m from ground
+       ============================================================ -->
+  <link name="base_laser">
+    <inertial>
+      <mass value="0.18"/>
+      <inertia ixx="0.001" ixy="0" ixz="0"
+               iyy="0.001" iyz="0" izz="0.001"/>
+    </inertial>
+    <visual>
+      <origin xyz="0 0 0" rpy="0 0 0"/>
+      <geometry>
+        <cylinder radius="${lidar_radius}" length="${lidar_length}"/>
+      </geometry>
+      <material name="black"/>
     </visual>
     <collision>
-      <origin xyz="0 0 ${chassis_height/2}"/>
-      <geometry>
-        <box size="${chassis_length} ${chassis_width} ${chassis_height}"/>
+      <origin xyz="0 0 0" rpy="0 0 0"/>
+      <geometry>
+        <cylinder radius="${lidar_radius}" length="${lidar_length}"/>
       </geometry>
     </collision>
-    <xacro:box_inertia m="${chassis_mass}"
-                       x="${chassis_length}"
-                       y="${chassis_width}"
-                       z="${chassis_height}"/>
-  </link>
-  <!-- ==================== DRIVE WHEELS ==================== -->
-  <xacro:drive_wheel name="left"  y_reflect="1"/>
-  <xacro:drive_wheel name="right" y_reflect="-1"/>
-  <!-- ==================== FRONT CASTER ==================== -->
-  <link name="front_caster_link">
-    <visual>
-      <geometry><sphere radius="${caster_radius}"/></geometry>
-      <material name="grey"><color rgba="0.5 0.5 0.5 1"/></material>
-    </visual>
-    <collision>
-      <geometry><sphere radius="${caster_radius}"/></geometry>
-    </collision>
-    <xacro:sphere_inertia m="${caster_mass}" r="${caster_radius}"/>
-  </link>
-  <joint name="front_caster_joint" type="fixed">
-    <parent link="base_link"/>
-    <child  link="front_caster_link"/>
-    <origin xyz="${chassis_length/2 - caster_radius} 0 ${-chassis_height/2 + caster_radius}"/>
-  </joint>
-  <!-- ==================== REAR CASTER ==================== -->
-  <link name="rear_caster_link">
-    <visual>
-      <geometry><sphere radius="${caster_radius}"/></geometry>
-      <material name="grey"><color rgba="0.5 0.5 0.5 1"/></material>
-    </visual>
-    <collision>
-      <geometry><sphere radius="${caster_radius}"/></geometry>
-    </collision>
-    <xacro:sphere_inertia m="${caster_mass}" r="${caster_radius}"/>
-  </link>
-  <joint name="rear_caster_joint" type="fixed">
-    <parent link="base_link"/>
-    <child  link="rear_caster_link"/>
-    <origin xyz="${-(chassis_length/2 - caster_radius)} 0 ${-chassis_height/2 + caster_radius}"/>
-  </joint>
-  <!-- ==================== LIDAR ==================== -->
-  <!-- base_laser is the agreed TF frame name from interfaces.md -->
-  <link name="base_laser">
-    <visual>
-      <geometry><cylinder radius="0.05" length="0.07"/></geometry>
-      <material name="black"><color rgba="0.1 0.1 0.1 1"/></material>
-    </visual>
-    <collision>
-      <geometry><cylinder radius="0.05" length="0.07"/></geometry>
-    </collision>
-    <inertial>
-      <mass value="0.1"/>
-      <inertia ixx="0.001" ixy="0" ixz="0" iyy="0.001" iyz="0" izz="0.001"/>
-    </inertial>
   </link>
   <joint name="lidar_joint" type="fixed">
     <parent link="base_link"/>
     <child  link="base_laser"/>
-    <!-- Mounted centered on top of chassis — clear 360 deg FOV -->
-    <origin xyz="0 0 ${chassis_height + lidar_z_offset}" rpy="0 0 0"/>
-  </joint>
-  <!-- ==================== CAMERA ==================== -->
+    <origin xyz="0 0 ${lidar_height}" rpy="0 0 0"/>
+  </joint>
+  <!-- ============================================================
+       IMU LINK
+       Mounted at center of chassis (on Pi)
+       [TUNE] Update xyz when IMU physical position is known
+       ============================================================ -->
+  <link name="imu_link">
+    <inertial>
+      <mass value="0.01"/>
+      <inertia ixx="0.00001" ixy="0" ixz="0"
+               iyy="0.00001" iyz="0" izz="0.00001"/>
+    </inertial>
+    <visual>
+      <origin xyz="0 0 0" rpy="0 0 0"/>
+      <geometry><box size="0.02 0.02 0.005"/></geometry>
+      <material name="grey"/>
+    </visual>
+  </link>
+  <joint name="imu_joint" type="fixed">
+    <parent link="base_link"/>
+    <child  link="imu_link"/>
+    <origin xyz="0 0 ${chassis_z}" rpy="0 0 0"/>
+  </joint>
+  <!-- ============================================================
+       CAMERA LINK (placeholder — update when camera selected)
+       ============================================================ -->
   <link name="camera_link">
-    <visual>
-      <geometry><box size="0.03 0.08 0.03"/></geometry>
-      <material name="black"><color rgba="0.1 0.1 0.1 1"/></material>
-    </visual>
-    <collision>
-      <geometry><box size="0.03 0.08 0.03"/></geometry>
-    </collision>
     <inertial>
       <mass value="0.05"/>
-      <inertia ixx="0.001" ixy="0" ixz="0" iyy="0.001" iyz="0" izz="0.001"/>
-    </inertial>
+      <inertia ixx="0.00001" ixy="0" ixz="0"
+               iyy="0.00001" iyz="0" izz="0.00001"/>
+    </inertial>
+    <visual>
+      <origin xyz="0 0 0" rpy="0 0 0"/>
+      <geometry><box size="0.03 0.09 0.03"/></geometry>
+      <material name="black"/>
+    </visual>
   </link>
   <joint name="camera_joint" type="fixed">
     <parent link="base_link"/>
     <child  link="camera_link"/>
-    <!-- Front face of chassis, mid-height -->
-    <origin xyz="${camera_x_offset} 0 ${chassis_height/2 + camera_z_offset}" rpy="0 0 0"/>
-  </joint>
-  <!-- Camera optical frame — Z forward, X right, Y down (ROS convention) -->
+    <!-- [TUNE] Update when camera mount position is finalized -->
+    <origin xyz="${chassis_length/2 - 0.01} 0 ${chassis_z + chassis_height/2}" rpy="0 0 0"/>
+  </joint>
   <link name="camera_optical_link"/>
   <joint name="camera_optical_joint" type="fixed">
@@ -180,31 +226,44 @@
     <origin xyz="0 0 0" rpy="${-pi/2} 0 ${-pi/2}"/>
   </joint>
-  <!-- ==================== GAZEBO PLUGINS ==================== -->
-  <!-- Differential drive controller -->
+  <!-- ============================================================
+       GAZEBO PLUGINS
+       ============================================================ -->
+  <!-- Differential drive plugin (skid steer — all 4 wheels) -->
   <gazebo>
     <plugin name="diff_drive" filename="libgazebo_ros_diff_drive.so">
-      <ros>
-        <namespace>/</namespace>
-      </ros>
-      <left_joint>left_wheel_joint</left_joint>
-      <right_joint>right_wheel_joint</right_joint>
-      <wheel_separation>${wheel_y_offset * 2}</wheel_separation>
-      <wheel_diameter>${wheel_radius * 2}</wheel_diameter>
+      <num_wheel_pairs>2</num_wheel_pairs>
+      <left_joint>front_left_wheel_joint</left_joint>
+      <left_joint>rear_left_wheel_joint</left_joint>
+      <right_joint>front_right_wheel_joint</right_joint>
+      <right_joint>rear_right_wheel_joint</right_joint>
+      <wheel_separation>${wheel_separation}</wheel_separation>
+      <wheel_diameter>${2*wheel_radius}</wheel_diameter>
       <max_wheel_torque>20</max_wheel_torque>
       <max_wheel_acceleration>1.0</max_wheel_acceleration>
-      <command_topic>cmd_vel</command_topic>
       <publish_odom>true</publish_odom>
       <publish_odom_tf>true</publish_odom_tf>
       <publish_wheel_tf>false</publish_wheel_tf>
-      <odometry_topic>odom</odometry_topic>
       <odometry_frame>odom</odometry_frame>
       <robot_base_frame>base_link</robot_base_frame>
-      <update_rate>30</update_rate>
     </plugin>
   </gazebo>
-  <!-- 2D LiDAR -->
+  <!-- IMU plugin -->
+  <gazebo reference="imu_link">
+    <sensor name="imu_sensor" type="imu">
+      <always_on>true</always_on>
+      <update_rate>50</update_rate>
+      <plugin filename="libgazebo_ros_imu_sensor.so" name="imu_plugin">
+        <topicName>/imu/data</topicName>
+        <bodyName>imu_link</bodyName>
+        <updateRateHZ>50.0</updateRateHZ>
+        <gaussianNoise>0.01</gaussianNoise>
+        <frameName>imu_link</frameName>
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
Commit message: Update camera and lidar frames

File: ros2_ws/src/description/urdf/warehouse_bot.urdf.xacro (robot description, xacro)
@@ -34,5 +34,5 @@
   <xacro:property name="wheelbase"       value="0.095"/>   <!-- front to rear axle, center to center -->
   <!-- LiDAR -->
-  <xacro:property name="lidar_height"    value="0.28"/>    <!-- from ground -->
+  <xacro:property name="lidar_height"    value="0.205"/>   <!-- from ground -->
   <xacro:property name="lidar_radius"    value="0.04"/>
   <xacro:property name="lidar_length"    value="0.06"/>
@@ -217,6 +217,6 @@
     <parent link="base_link"/>
     <child  link="camera_link"/>
-    <!-- [TUNE] Update when camera mount position is finalized -->
-    <origin xyz="${chassis_length/2 - 0.01} 0 ${chassis_z + chassis_height/2}" rpy="0 0 0"/>
+    <!-- Camera is centered left/right, 10 cm forward of robot center, 8.5 cm from ground. -->
+    <origin xyz="0.10 0 0.085" rpy="0 0 0"/>
   </joint>
   <link name="camera_optical_link"/>
